File: ev-charger-met16/ev-charger-met16.sch (KiCad schematic (older format))
At the start: 62 parts, among them J1 Screw_Terminal_01x02, J10 Conn_02x02_Counter_Clockwise, J2 Conn_01x03, J3 Conn_01x15, J4 Conn_01x15, J5 Lusterklemme-6mm2-40A, J6 Lusterklemme-6mm2-40A, J7 LCD-Sure, J8 UART-Harwin4, J9 Conn_01x03, Q1 NTR2101P, Q2 MMBF170, Q3 NTR2101P, Q4 MMBF170, SW1 SW_PT65-501, SW2 SW_DPDT_x2, U1 ARDUINO-NANO, U2 HLK-PM01, U3 ebay-253052736386, U4 ACS712, U5 ebay-232542976388

Commit message: Erster Entwurf V0.2
Parts:
- removed Q1, Q3: NTR2101P, TO_SOT_Packages_SMD:SOT-23_Handsoldering, symbol NTR2101P
- removed Q2, Q4: MMBF170, TO_SOT_Packages_SMD:SOT-23_Handsoldering, symbol MMBF170
- removed R1: 15k, Resistors_SMD:R_1206_HandSoldering, symbol R
- removed R2, R3: 10k, Resistors_SMD:R_1206_HandSoldering, symbol R
- removed R4: 33k, Resistors_SMD:R_1206_HandSoldering, symbol R
- removed R6: 1k, Resistors_SMD:R_1206_HandSoldering, symbol R
- removed R7: 47k, Resistors_SMD:R_1206_HandSoldering, symbol R
- removed U5: ebay-232542976388, MyFootprints:ebay-232542976388, symbol ebay-232542976388
- added C12: 22n, Capacitors_SMD:C_1206_HandSoldering, symbol C
- added R31: 1k, Resistors_SMD:R_1206_HandSoldering, symbol R
- added R32: 10k, Resistors_SMD:R_1206_HandSoldering, symbol R
- added U6: AD822, Housings_SOIC:SO-8_5.3x6.2mm_Pitch1.27mm, symbol AD822
- J1: footprint MyFootprints:Terminalblock-2x-5mm -> Project:Terminalblock-2x-5mm
- J5: footprint MyFootprints:Lusterklemme-PA30P-6mm2-40A-x3-N -> Project:Lusterklemme-PA30P-6mm2-40A-x3-N
- J6: footprint MyFootprints:Lusterklemme-PA30P-6mm2-40A-x3-S -> Project:Lusterklemme-PA30P-6mm2-40A-x3-S
- J7: footprint MyFootprints:LCD-Sure-shifted-064 -> Project:LCD-Sure-shifted-064
- R33: renamed from R8; value 12k -> 100k
- R38: renamed from R9; value 1k -> 10k
- RV2: renamed from RV1; footprint Potentiometers:Potentiometer_Trimmer_Bourns_3299W -> Potentiometers:Potentiometer_Trimmer_Bourns_3296W
- SW1: footprint MyFootprints:SW_DIP_x3_W7.62mm_PT65-501 -> Project:SW_DIP_x3_W7.62mm_PT65-501
- U1: footprint MyFootprints:Arduino-Nano -> Project:Arduino-Nano
- U2: footprint MyFootprints:HLK_PM01 -> Project:HLK_PM01
- U3: footprint MyFootprints:ebay-253052736386 -> Project:ebay-253052736386
- renumbered C3 to C10, C5 to C11, C2 to C7, C1 to C8, C4 to C9, R12 to R29, R11 to R30
Connections:
- wire segments 246 -> 241
- no-connect marks 3 -> 5
Other:
- moved on the sheet: C8, D1, R10, R33, R38, R5

Commit message: V0.2 Design finished
Parts:
- added R34, R35: 10k, Resistors_SMD:R_1206_HandSoldering, symbol R
- C8: footprint Capacitors_SMD:C_1210_HandSoldering -> Capacitors_SMD:C_1206_HandSoldering
- R32: value 10k -> 22k
Connections:
- wire segments 241 -> 245
Changed lines of the file:
@@
 F 0 "C8" H 9625 2850 50  0000 L CNN
 F 1 "1u" H 9625 2650 50  0000 L CNN
-F 2 "Capacitors_SMD:C_1210_HandSoldering" H 9638 2600 50  0001 C CNN
+F 2 "Capacitors_SMD:C_1206_HandSoldering" H 9638 2600 50  0001 C CNN
 F 3 "" H 9600 2750 50  0001 C CNN
 	1    9600 2750
@@
 P 6750 1100
 F 0 "R32" V 6830 1100 50  0000 C CNN
-F 1 "10k" V 6750 1100 50  0000 C CNN
+F 1 "22k" V 6750 1100 50  0000 C CNN
 F 2 "Resistors_SMD:R_1206_HandSoldering" V 6680 1100 50  0001 C CNN
 F 3 "" H 6750 1100 50  0001 C CNN
@@
 $EndComp
 $Comp
-L -12V #PWR25
+L -12V #PWR26
 U 1 1 5AF95D4C
 P 6700 2250
-F 0 "#PWR25" H 6700 2350 50  0001 C CNN
+F 0 "#PWR26" H 6700 2350 50  0001 C CNN
 F 1 "-12V" H 6700 2400 50  0000 C CNN
 F 2 "" H 6700 2250 50  0001 C CNN
@@
 L GND #PWR040
 U 1 1 5AF968E9
-P 6400 2100
-F 0 "#PWR040" H 6400 1850 50  0001 C CNN
-F 1 "GND" H 6400 1950 50  0000 C CNN
-F 2 "" H 6400 2100 50  0001 C CNN
-F 3 "" H 6400 2100 50  0001 C CNN
-	1    6400 2100
-	1    0    0    -1
-$EndComp
-Wire Wire Line
-	6400 2100 6400 2000
-Wire Wire Line
-	6400 2000 6500 2000
+P 6150 2900
+F 0 "#PWR040" H 6150 2650 50  0001 C CNN
+F 1 "GND" H 6150 2750 50  0000 C CNN
+F 2 "" H 6150 2900 50  0001 C CNN
+F 3 "" H 6150 2900 50  0001 C CNN
+	1    6150 2900
+	1    0    0    -1
+$EndComp
 Wire Wire Line
 	6350 1800 6500 1800
@@
 $EndComp
 $Comp
-L -12V #PWR27
+L -12V #PWR28
 U 1 1 5AF9BD9F
 P 7100 1600
-F 0 "#PWR27" H 7100 1700 50  0001 C CNN
+F 0 "#PWR28" H 7100 1700 50  0001 C CNN
 F 1 "-12V" H 7100 1750 50  0000 C CNN
 F 2 "" H 7100 1600 50  0001 C CNN
@@
 Connection ~ 7400 3750
 Connection ~ 7300 4650
+$Comp
+L R R35
+U 1 1 5AFBC6D4
+P 6150 2700
+F 0 "R35" V 6230 2700 50  0000 C CNN
+F 1 "10k" V 6150 2700 50  0000 C CNN
+F 2 "Resistors_SMD:R_1206_HandSoldering" V 6080 2700 50  0001 C CNN
+F 3 "" H 6150 2700 50  0001 C CNN
+	1    6150 2700
+	1    0    0    -1
+$EndComp
+$Comp
+L R R34
+U 1 1 5AFBC7E3
+P 6150 2300
+F 0 "R34" V 6230 2300 50  0000 C CNN
+F 1 "10k" V 6150 2300 50  0000 C CNN
+F 2 "Resistors_SMD:R_1206_HandSoldering" V 6080 2300 50  0001 C CNN
+F 3 "" H 6150 2300 50  0001 C CNN
+	1    6150 2300
+	1    0    0    -1
+$EndComp
+$Comp
+L +5V #PWR042
+U 1 1 5AFBCEAD
+P 6150 2100
+F 0 "#PWR042" H 6150 1950 50  0001 C CNN
+F 1 "+5V" H 6150 2240 50  0000 C CNN
+F 2 "" H 6150 2100 50  0001 C CNN
+F 3 "" H 6150 2100 50  0001 C CNN
+	1    6150 2100
+	1    0    0    -1
+$EndComp
+Wire Wire Line
+	6150 2900 6150 2850
+Wire Wire Line
+	6150 2550 6150 2450
+Wire Wire Line
+	6150 2150 6150 2100
+Wire Wire Line
+	6150 2500 6400 2500
+Wire Wire Line
+	6400 2500 6400 2000
+Wire Wire Line
+	6400 2000 6500 2000
+Connection ~ 6150 2500
 $EndSCHEMATC
