File: ev-charger-met16/ev-charger-met16.sch (KiCad schematic (older format))
At the start: 57 parts, among them J1 Screw_Terminal_01x02, J10 Conn_02x02_Counter_Clockwise, J2 Conn_01x03, J3 Conn_01x15, J4 Conn_01x15, J5 Lusterklemme-6mm2-40A, J6 Lusterklemme-6mm2-40A, J7 LCD-Sure, J8 UART-Harwin4, J9 Conn_01x03, SW1 SW_PT65-501, SW2 SW_DPDT_x2, U1 ARDUINO-NANO, U2 HLK-PM01, U3 ebay-253052736386, U4 ACS712, U6 AD822

Commit message: Version V0.2 - ready for multi-cb
Parts:
- D1, D4, D5: footprint Diodes_SMD:D_SOD-323_HandSoldering -> Diodes_SMD:D_SMA_Handsoldering
Changed lines of the file:
@@
 Sheet 1 2
 Title "EV Charger Metal 16A"
-Date "2018-04-02"
-Rev "V1.0"
+Date "2018-05-27"
+Rev "V0.2"
 Comp "Manfred Steiner"
-Comment1 ""
+Comment1 "First Prototype"
 Comment2 ""
 Comment3 ""
@@
 F 0 "D1" H 9050 2400 50  0000 C CNN
 F 1 "D_Schottky" H 9000 2600 50  0001 C CNN
-F 2 "Diodes_SMD:D_SOD-323_HandSoldering" H 9050 2500 50  0001 C CNN
+F 2 "Diodes_SMD:D_SMA_Handsoldering" H 9050 2500 50  0001 C CNN
 F 3 "" H 9050 2500 50  0001 C CNN
 	1    9050 2500
@@
 F 0 "D4" H 1400 1800 50  0000 C CNN
 F 1 "D_Schottky" H 1350 2000 50  0001 C CNN
-F 2 "Diodes_SMD:D_SOD-323_HandSoldering" H 1400 1900 50  0001 C CNN
+F 2 "Diodes_SMD:D_SMA_Handsoldering" H 1400 1900 50  0001 C CNN
 F 3 "" H 1400 1900 50  0001 C CNN
 	1    1400 1900
@@
 F 0 "D5" H 8550 750 50  0000 C CNN
 F 1 "D_Schottky" H 8500 950 50  0001 C CNN
-F 2 "Diodes_SMD:D_SOD-323_HandSoldering" H 8550 850 50  0001 C CNN
+F 2 "Diodes_SMD:D_SMA_Handsoldering" H 8550 850 50  0001 C CNN
 F 3 "" H 8550 850 50  0001 C CNN
 	1    8550 850
