File: ev-charger-met16/ev-charger-met16.kicad_pcb (KiCad board)
At the start: 2 copper layers, 165 x 70 mm, 70 parts, among them J1 Screw_Terminal_01x02, J10 Conn_02x02_Counter_Clockwise, J2 Conn_01x03, J3 Conn_01x15, J4 Conn_01x15, J5 Lusterklemme-6mm2-40A, J6 Lusterklemme-6mm2-40A, J7 LCD-Sure, J8 UART-Harwin4, J9 Conn_01x03, Q1 NTR2101P, Q2 MMBF170, Q3 NTR2101P, Q4 MMBF170, SW1 SW_PT65-501, SW2 SW_DPDT_x2, U1 ARDUINO-NANO, U2 HLK-PM01, U3 ebay-253052736386, U4 ACS712, U5 ebay-232542976388

Commit message: Erster Entwurf V0.2
Parts:
- removed Q1, Q3: NTR2101P, TO_SOT_Packages_SMD:SOT-23_Handsoldering
- removed Q2, Q4: MMBF170, TO_SOT_Packages_SMD:SOT-23_Handsoldering
- added C1: 1nF, Capacitors_SMD:C_1206_HandSoldering, F.Cu at (129.8, 87.8)
- added C12: 22n, Capacitors_SMD:C_1206_HandSoldering, F.Cu at (126.2, 64.8)
- added C2: 1uF, Capacitors_SMD:C_1206_HandSoldering, B.Cu at (115.3, 84.3)
- added C3: 1nF, Capacitors_SMD:C_1206_HandSoldering, F.Cu at (150.9, 88.1)
- added C4: 1uF, Capacitors_SMD:C_1206_HandSoldering, F.Cu at (127.1, 85.7)
- added C5: 22nF, Capacitors_SMD:C_1206_HandSoldering, F.Cu at (143.0, 94.2)
- added R11: 100, Resistors_SMD:R_1206_HandSoldering, B.Cu at (112.8, 84.3)
- added R12: 820k, Resistors_SMD:R_1206_HandSoldering, B.Cu at (98.8, 78.0)
- added R31: 1k, Resistors_SMD:R_1206_HandSoldering, F.Cu at (139.2, 75.7)
- added R32: 10k, Resistors_SMD:R_1206_HandSoldering, F.Cu at (129.5, 76.2)
- added R8: 10k, Resistors_SMD:R_1206_HandSoldering, B.Cu at (118.1, 72.4)
- added R9: 100k, Resistors_SMD:R_1206_HandSoldering, F.Cu at (153.4, 88.1)
- added RV2: 10K, Potentiometers:Potentiometer_Trimmer_Bourns_3296W, F.Cu at (180.8, 60.2)
- added T1: Transformer_1P_1S, Project:Transformer-zmpt101b_ebay-121438904988, F.Cu at (109.7, 84.1)
- added U6: AD822, Housings_SOIC:SO-8_5.3x6.2mm_Pitch1.27mm, F.Cu at (131.1, 69.3)
- J1: footprint MyFootprints:Terminalblock-2x-5mm -> Project:Terminalblock-2x-5mm
- J5: footprint MyFootprints:Lusterklemme-PA30P-6mm2-40A-x3-N -> Project:Lusterklemme-PA30P-6mm2-40A-x3-N
- J6: footprint MyFootprints:Lusterklemme-PA30P-6mm2-40A-x3-S -> Project:Lusterklemme-PA30P-6mm2-40A-x3-S
- R1: value 15k -> 100k
- R2, R3: moved to B.Cu
- R33: renamed from R8; value 12k -> 100k
- R38: renamed from R9; value 1k -> 10k
- R4: value 33k -> 10k
- R6: value 1k -> 10k
- R7: value 47k -> 10k
- RV1: value 10K -> 10k; footprint Potentiometers:Potentiometer_Trimmer_Bourns_3299W -> Potentiometers:Potentiometer_Trimmer_Bourns_3296W
- SW1: footprint MyFootprints:SW_DIP_x3_W7.62mm_PT65-501 -> Project:SW_DIP_x3_W7.62mm_PT65-501
- U1: footprint MyFootprints:Arduino-Nano -> Project:Arduino-Nano
- U2: footprint MyFootprints:HLK_PM01 -> Project:HLK_PM01
- U3: footprint MyFootprints:ebay-253052736386 -> Project:ebay-253052736386
- U5: value ebay-232542976388 -> LM358; footprint MyFootprints:ebay-232542976388 -> Housings_SOIC:SO-8_5.3x6.2mm_Pitch1.27mm
- moved RV1 65.1 mm to (122.9, 89.9), turned to 270 degrees
- moved R4 35.7 mm to (143.0, 91.7), turned to 180 degrees
- moved U5 34.2 mm to (144.0, 86.9), turned to 180 degrees
- moved R25 34.0 mm to (168.4, 90.2), turned to 90 degrees
- moved J9 30.8 mm to (155.4, 95.2), turned to 270 degrees
- moved D1 29.2 mm to (131.3, 62.7), turned to 180 degrees
- moved R6 24.4 mm to (129.4, 81.2)
- moved R10 21.3 mm to (182.6, 75.2)
- moved R33 20.5 mm to (139.2, 66.8)
- moved R7 19.5 mm to (139.2, 81.8), turned to 0 degrees
- moved R5 18.7 mm to (139.2, 78.2), turned to 180 degrees
- moved R38 17.5 mm to (136.7, 66.8), turned to 270 degrees
- moved R29 16.1 mm to (165.6, 90.2), turned to 90 degrees
- moved C8 15.1 mm to (179.8, 76.5), turned to 270 degrees
- moved R1 14.9 mm to (132.3, 87.8)
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- renumbered C3 to C10, C5 to C11, C2 to C7, C1 to C8, C4 to C9, R12 to R29, R11 to R30
Connections:
- C11 pad 1: /A2 -> /A1
- C8 pad 1: /A0 -> /A6
- C9 pad 1: /A1 -> /A0
- D1 pad 1: /A0 -> /A6
- R1 pad 1: Net-(Q1-Pad3) -> Net-(C1-Pad1)
- R1 pad 2: Net-(Q4-Pad1) -> Net-(C1-Pad2)
- R10 pad 1: /A0 -> /A6
- R13 pad 1: /A1 -> /A0
- R2 pad 1: Net-(Q4-Pad1) -> Net-(C1-Pad2)
- R2 pad 2: -12V -> Net-(C2-Pad1)
- R21 pad 2: /A6 -> /A2
- R22 pad 2: /A6 -> /A2
- R25 pad 2: /A2 -> /A1
- R26 pad 1: /A2 -> /A1
- R29 pad 2: /A1 -> /A0
- R3 pad 1: Net-(Q3-Pad1) -> Net-(R3-Pad1)
- R3 pad 2: +12V -> Net-(R11-Pad1)
- R33 pad 2: Net-(D1-Pad2) -> Net-(R33-Pad2)
- R38 pad 1: Net-(D1-Pad2) -> Net-(R33-Pad2)
- R4 pad 1: Net-(Q3-Pad1) -> Net-(R4-Pad1)
- R4 pad 2: Net-(Q2-Pad3) -> +5V
- R5 pad 1: Net-(Q3-Pad3) -> /CP
- R5 pad 2: /CP -> Net-(R32-Pad2)
- R6 pad 1: /CP -> Net-(C3-Pad2)
- R7 pad 1: PWM -> GND
- R7 pad 2: +5V -> Net-(R4-Pad1)
- RV1 pad 1: +5V -> Net-(C1-Pad1)
- RV1 pad 2: /VEE -> Net-(C4-Pad2)
- U5 pad 1: GND -> /MVOLT
- U5 pad 2: GND -> Net-(C3-Pad2)
- U5 pad 3: /MVOLT -> Net-(R4-Pad1)
- U5 pad 4: +5V -> GND
- U5 pad 5: /NOUT -> Net-(R3-Pad1)
- U5 pad 6: /L -> Net-(C1-Pad2)
Routing:
- net Net-(Q3-Pad3): track 55.4 -> 0.00 mm, vias 4 -> 0
- net Net-(C4-Pad1): track 44.4 -> 2.69 mm, vias 4 -> 0
- net PWM: track 74.4 -> 39.8 mm, vias 3 -> 1
- net Net-(R3-Pad1): track 0.00 -> 32.8 mm, vias 0 -> 1
- net Net-(C3-Pad2): track 0.00 -> 31.4 mm
- net +12V: track 41.0 -> 10.8 mm
- net Net-(C1-Pad2): track 0.00 -> 25.1 mm, vias 0 -> 1
- net /CP: track 64.3 -> 86.7 mm
- net /NOUT: track 20.7 -> 0.00 mm
- net Net-(C1-Pad1): track 0.00 -> 18.8 mm
- net GND: track 48.6 -> 65.0 mm, vias 8 -> 10
- net Net-(R4-Pad1): track 0.00 -> 16.2 mm
- net /MVOLT: track 16.3 -> 31.9 mm
- net Net-(Q2-Pad3): track 15.3 -> 0.00 mm
- net Net-(R32-Pad2): track 0.00 -> 15.2 mm
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Other:
- board text added: "EV Charger MET16 V0.2? / SX"
- board text removed: "EV Charger MET16 V0.1 / SX"

Commit message: V0.2 Design finished
Parts:
- added R34: 10k, Resistors_SMD:R_1206_HandSoldering, F.Cu at (146.6, 67.1)
- added R35: 10k, Resistors_SMD:R_1206_HandSoldering, F.Cu at (144.0, 67.0)
- C8: footprint Capacitors_SMD:C_1210_HandSoldering -> Capacitors_SMD:C_1206_HandSoldering
- R32: value 10k -> 22k
- moved R5 6.62 mm to (132.6, 78.7)
- moved R6 5.64 mm to (134.9, 82.5)
- moved R7 5.34 mm to (144.5, 82.0), turned to 180 degrees
- moved R22 4.83 mm to (149.1, 67.1)
- moved R32 1.52 mm to (131.1, 76.2)
- moved U5 0.76 mm to (143.3, 86.8)
- moved R14 0.76 mm to (175.8, 77.0)
- moved R15 0.76 mm to (173.2, 77.0)
- moved C8 0.57 mm to (180.1, 77.0), turned to 90 degrees
- moved C3 0.51 mm to (150.4, 88.1)
- moved R9 0.51 mm to (152.9, 88.1)
- moved R31 0.51 mm to (139.2, 76.2)
- moved R10 0.25 mm to (182.6, 75.4)
- moved R11 0.25 mm to (113.0, 84.3)
- moved R3 0.25 mm to (114.0, 74.4)
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Connections:
- J8 pad 1: GND -> Net-(D4-Pad2)
- J8 pad 2: Net-(D4-Pad2) -> GND
- U6 pad 2: GND -> Net-(R34-Pad2)
Routing:
- net /PE: track 11.4 -> 57.7 mm
- net GND: track 65.0 -> 89.5 mm, vias 10 -> 7
- net Net-(R34-Pad2): track 0.00 -> 22.5 mm, vias 0 -> 2
- net Net-(R32-Pad2): track 15.2 -> 6.50 mm
- net /CP: track 86.7 -> 92.0 mm
- net Net-(C3-Pad2): track 31.4 -> 26.8 mm
- net Net-(C4-Pad1): track 2.69 -> 6.23 mm
- net /D3: track 53.5 -> 50.8 mm
- net LCD-RS: track 133.4 -> 131.3 mm
- net /A6: track 73.5 -> 75.5 mm
- net Net-(R4-Pad1): track 16.2 -> 14.5 mm
- net +5V: track 170.8 -> 172.3 mm
- net Net-(R3-Pad1): track 32.8 -> 31.6 mm
- net /A7: track 76.3 -> 75.2 mm
- net Net-(R31-Pad2): track 9.09 -> 8.06 mm
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Other:
- net class 230V added: clearance 1.5, trace_width 1, via_dia 1, via_drill 0.8
- net class PE added: clearance 1, trace_width 1, via_dia 1, via_drill 0.8

Commit message: Version V0.2 - ready for multi-cb
Parts:
- D1, D4, D5: footprint Diodes_SMD:D_SOD-323_HandSoldering -> Diodes_SMD:D_SMA_Handsoldering
- moved D5 4.58 mm to (205.5, 86.1)
- moved R8 4.06 mm to (114.0, 72.1), turned to 0 degrees
- moved D4 3.18 mm to (202.4, 65.2)
- moved R2 2.54 mm to (120.4, 80.5)
- moved C12 2.03 mm to (126.2, 66.8)
- moved U3 2.00 mm to (102.0, 67.0)
- moved D2 0.97 mm to (205.5, 61.5)
- moved D1 0.92 mm to (131.8, 62.0)
- moved D3 0.66 mm to (205.5, 57.7)
- moved R17 0.51 mm to (128.5, 59.4)
- moved SW2 0.48 mm to (205.2, 81.8)
- moved SW1 0.44 mm to (200.4, 70.0)
Routing:
- net /NOUT: track 0.00 -> 14.9 mm
- net /N: track 46.8 -> 61.7 mm
- net +5V: track 172.3 -> 163.0 mm
- net Net-(D5-Pad1): track 10.1 -> 6.41 mm
- net /D5: track 42.6 -> 40.0 mm
- net Net-(C1-Pad2): track 24.3 -> 21.9 mm
- net GND: track 89.5 -> 91.6 mm
- net Net-(D4-Pad2): track 5.04 -> 6.36 mm
- net Net-(C2-Pad1): track 5.64 -> 4.34 mm
- net -12V: track 20.5 -> 19.3 mm
- net +12V: track 10.8 -> 12.0 mm
- net /A5: track 33.5 -> 34.6 mm
- net Net-(R3-Pad1): track 31.6 -> 32.7 mm
- net /D2: track 22.5 -> 21.5 mm
Other:
- net class PE: clearance 1 -> 0.3
- board text added: "EV Charger MET16 V0.2 / SX"
- board text removed: "EV Charger MET16 V0.2? / SX"
