File: rpi-atmega324-modbus-gateway-min/MODBUS.sch (KiCad schematic (older format))
At the start: 40 parts, among them J10 Conn_01x02, J11 Conn_01x02, J12 Conn_01x02, J13 Conn_01x02, J14 Screw_Terminal_01x02, J15 Screw_Terminal_01x02, J6 Conn_01x03, J7 Conn_01x03, J8 Conn_01x02, J9 Conn_01x02, U2 SN65HVD11, U3 SN65HVD11

Commit message: Modbus Gateway V0.1 - Tapeout 1
Parts:
- U2, U3: footprint Housings_SOIC:SOIC-8_3.9x4.9mm_Pitch1.27mm -> Project:SOIC-8_3.9x4.9mm_Pitch1.27mm_Handsolded
Changed lines of the file:
@@
 LIBS:contrib
 LIBS:valves
-LIBS:raspberry
-LIBS:terminals
 LIBS:sx-atmega
+LIBS:sx-raspberry
+LIBS:sx-terminals
 LIBS:rpi-atmega324-modbus-gateway-min-cache
 EELAYER 25 0
@@
 F 0 "U2" H 3910 2550 50  0000 C CNN
 F 1 "SN65HVD11" H 4180 2550 50  0000 L CNN
-F 2 "Housings_SOIC:SOIC-8_3.9x4.9mm_Pitch1.27mm" H 4150 1400 50  0001 C CNN
+F 2 "Project:SOIC-8_3.9x4.9mm_Pitch1.27mm_Handsolded" H 4150 1400 50  0001 C CNN
 F 3 "" H 4150 2150 50  0001 C CNN
 	1    4150 2100
@@
 $EndComp
 $Comp
-L GND #PWR019
+L GND #PWR022
 U 1 1 5B141CE2
 P 4150 2750
-F 0 "#PWR019" H 4150 2500 50  0001 C CNN
+F 0 "#PWR022" H 4150 2500 50  0001 C CNN
 F 1 "GND" H 4150 2600 50  0000 C CNN
 F 2 "" H 4150 2750 50  0001 C CNN
@@
 $EndComp
 $Comp
-L +3V3 #PWR020
+L +3V3 #PWR023
 U 1 1 5B142EF2
 P 3600 1500
-F 0 "#PWR020" H 3600 1350 50  0001 C CNN
+F 0 "#PWR023" H 3600 1350 50  0001 C CNN
 F 1 "+3V3" H 3600 1640 50  0000 C CNN
 F 2 "" H 3600 1500 50  0001 C CNN
@@
 $EndComp
 $Comp
-L +3V3 #PWR021
+L +3V3 #PWR024
 U 1 1 5B142F69
 P 4150 1300
-F 0 "#PWR021" H 4150 1150 50  0001 C CNN
+F 0 "#PWR024" H 4150 1150 50  0001 C CNN
 F 1 "+3V3" H 4150 1440 50  0000 C CNN
 F 2 "" H 4150 1300 50  0001 C CNN
@@
 $EndComp
 $Comp
-L GND #PWR022
+L GND #PWR025
 U 1 1 5B143126
 P 3500 2800
-F 0 "#PWR022" H 3500 2550 50  0001 C CNN
+F 0 "#PWR025" H 3500 2550 50  0001 C CNN
 F 1 "GND" H 3500 2650 50  0000 C CNN
 F 2 "" H 3500 2800 50  0001 C CNN
@@
 $EndComp
 $Comp
-L GND #PWR023
+L GND #PWR026
 U 1 1 5B1431C9
 P 2850 3200
-F 0 "#PWR023" H 2850 2950 50  0001 C CNN
+F 0 "#PWR026" H 2850 2950 50  0001 C CNN
 F 1 "GND" H 2850 3050 50  0000 C CNN
 F 2 "" H 2850 3200 50  0001 C CNN
@@
 $EndComp
 $Comp
-L GND #PWR024
+L GND #PWR027
 U 1 1 5B143233
 P 7350 2150
-F 0 "#PWR024" H 7350 1900 50  0001 C CNN
+F 0 "#PWR027" H 7350 1900 50  0001 C CNN
 F 1 "GND" H 7350 2000 50  0000 C CNN
 F 2 "" H 7350 2150 50  0001 C CNN
@@
 $EndComp
 $Comp
-L GND #PWR025
+L GND #PWR028
 U 1 1 5B1432E2
 P 4950 1500
-F 0 "#PWR025" H 4950 1250 50  0001 C CNN
+F 0 "#PWR028" H 4950 1250 50  0001 C CNN
 F 1 "GND" H 4950 1350 50  0000 C CNN
 F 2 "" H 4950 1500 50  0001 C CNN
@@
 $EndComp
 $Comp
-L +3V3 #PWR026
+L +3V3 #PWR029
 U 1 1 5B1450DC
 P 6650 1050
-F 0 "#PWR026" H 6650 900 50  0001 C CNN
+F 0 "#PWR029" H 6650 900 50  0001 C CNN
 F 1 "+3V3" H 6650 1190 50  0000 C CNN
 F 2 "" H 6650 1050 50  0001 C CNN
@@
 $EndComp
 $Comp
-L GND #PWR027
+L GND #PWR030
 U 1 1 5B145265
 P 6400 3250
-F 0 "#PWR027" H 6400 3000 50  0001 C CNN
+F 0 "#PWR030" H 6400 3000 50  0001 C CNN
 F 1 "GND" H 6400 3100 50  0000 C CNN
 F 2 "" H 6400 3250 50  0001 C CNN
@@
 F 0 "U3" H 3910 5650 50  0000 C CNN
 F 1 "SN65HVD11" H 4180 5650 50  0000 L CNN
-F 2 "Housings_SOIC:SOIC-8_3.9x4.9mm_Pitch1.27mm" H 4150 4500 50  0001 C CNN
+F 2 "Project:SOIC-8_3.9x4.9mm_Pitch1.27mm_Handsolded" H 4150 4500 50  0001 C CNN
 F 3 "" H 4150 5250 50  0001 C CNN
 	1    4150 5200
@@
 $EndComp
 $Comp
-L GND #PWR028
+L GND #PWR031
 U 1 1 5B14B378
 P 4150 5850
-F 0 "#PWR028" H 4150 5600 50  0001 C CNN
+F 0 "#PWR031" H 4150 5600 50  0001 C CNN
 F 1 "GND" H 4150 5700 50  0000 C CNN
 F 2 "" H 4150 5850 50  0001 C CNN
@@
 $EndComp
 $Comp
-L +3V3 #PWR029
+L +3V3 #PWR032
 U 1 1 5B14B3B2
 P 3600 4600
-F 0 "#PWR029" H 3600 4450 50  0001 C CNN
+F 0 "#PWR032" H 3600 4450 50  0001 C CNN
 F 1 "+3V3" H 3600 4740 50  0000 C CNN
 F 2 "" H 3600 4600 50  0001 C CNN
@@
 $EndComp
 $Comp
-L +3V3 #PWR030
+L +3V3 #PWR033
 U 1 1 5B14B3B8
 P 4150 4400
-F 0 "#PWR030" H 4150 4250 50  0001 C CNN
+F 0 "#PWR033" H 4150 4250 50  0001 C CNN
 F 1 "+3V3" H 4150 4540 50  0000 C CNN
 F 2 "" H 4150 4400 50  0001 C CNN
@@
 $EndComp
 $Comp
-L GND #PWR031
+L GND #PWR034
 U 1 1 5B14B3C4
 P 3500 5900
-F 0 "#PWR031" H 3500 5650 50  0001 C CNN
+F 0 "#PWR034" H 3500 5650 50  0001 C CNN
 F 1 "GND" H 3500 5750 50  0000 C CNN
 F 2 "" H 3500 5900 50  0001 C CNN
@@
 $EndComp
 $Comp
-L GND #PWR032
+L GND #PWR035
 U 1 1 5B14B3CA
 P 2850 6300
-F 0 "#PWR032" H 2850 6050 50  0001 C CNN
+F 0 "#PWR035" H 2850 6050 50  0001 C CNN
 F 1 "GND" H 2850 6150 50  0000 C CNN
 F 2 "" H 2850 6300 50  0001 C CNN
@@
 $EndComp
 $Comp
-L GND #PWR033
+L GND #PWR036
 U 1 1 5B14B3D0
 P 7400 5250
-F 0 "#PWR033" H 7400 5000 50  0001 C CNN
+F 0 "#PWR036" H 7400 5000 50  0001 C CNN
 F 1 "GND" H 7400 5100 50  0000 C CNN
 F 2 "" H 7400 5250 50  0001 C CNN
@@
 $EndComp
 $Comp
-L GND #PWR034
+L GND #PWR037
 U 1 1 5B14B3D6
 P 4950 4600
-F 0 "#PWR034" H 4950 4350 50  0001 C CNN
+F 0 "#PWR037" H 4950 4350 50  0001 C CNN
 F 1 "GND" H 4950 4450 50  0000 C CNN
 F 2 "" H 4950 4600 50  0001 C CNN
@@
 $EndComp
 $Comp
-L +3V3 #PWR035
+L +3V3 #PWR038
 U 1 1 5B14B412
 P 6650 4150
-F 0 "#PWR035" H 6650 4000 50  0001 C CNN
+F 0 "#PWR038" H 6650 4000 50  0001 C CNN
 F 1 "+3V3" H 6650 4290 50  0000 C CNN
 F 2 "" H 6650 4150 50  0001 C CNN
@@
 $EndComp
 $Comp
-L GND #PWR036
+L GND #PWR039
 U 1 1 5B14B41E
 P 6400 6350
-F 0 "#PWR036" H 6400 6100 50  0001 C CNN
+F 0 "#PWR039" H 6400 6100 50  0001 C CNN
 F 1 "GND" H 6400 6200 50  0000 C CNN
 F 2 "" H 6400 6350 50  0001 C CNN
