File: rpi-atmega324-modbus-gateway-min/rpi-atmega324-modbus-gateway-min.kicad_pcb (KiCad board)
At the start: 2 copper layers, 68 x 64.4 mm, 66 parts, among them J1 Raspberry_Pi_2+, J10 Conn_01x02, J11 Conn_01x02, J12 Conn_01x02, J13 Conn_01x02, J14 Screw_Terminal_01x02, J15 Screw_Terminal_01x02, J16 Conn_01x11, J17 Conn_01x11, J18 Conn_01x11, J19 Conn_01x11, J2 UART-Harwin4, J3 Conn_01x02, J4 Conn_02x03_Odd_Even, J5 Atmega-ISP-6, J6 Conn_01x03, J7 Conn_01x03, J8 Conn_01x02, J9 Conn_01x02, SW1 SW_Push, U1 ATMEGA324P-20AU, U2 SN65HVD11, U3 SN65HVD11, Y1 12MHz

Commit message: Modbus Gateway V0.1 - Tapeout 1
Parts:
- added D7: LED, LEDs:LED_0805_HandSoldering, F.Cu at (157.2, 58.9)
- added D8: LED, LEDs:LED_0805_HandSoldering, F.Cu at (154.7, 58.9)
- added D9: LED, LEDs:LED_0805_HandSoldering, F.Cu at (152.1, 58.9)
- added R27: 560R, Resistors_SMD:R_1206_HandSoldering, B.Cu at (151.1, 66.0)
- added R28: 560R, Resistors_SMD:R_1206_HandSoldering, B.Cu at (151.1, 57.9)
- added R29: 560R, Resistors_SMD:R_1206_HandSoldering, B.Cu at (148.6, 55.4)
- added SW2: SW_SPST, Project:SW-ebay-171865305033, F.Cu at (153.7, 53.3)
- J2: value UART-Harwin4 -> UART-Harwin3; footprint Connectors_Harwin:Harwin_LTek-Male_04x2.00mm_Straight_StrainRelief -> Connectors_Harwin:Harwin_LTek-Male_03x2.00mm_Straight_StrainRelief
- J4: footprint Pin_Headers:Pin_Header_Straight_2x03_Pitch2.54mm -> Project:Jumper_3x_2x03_Pitch2.54mm
- R5: moved to B.Cu
- U1: footprint Housings_QFP:TQFP-44_10x10mm_Pitch0.8mm -> Project:TQFP-44_10x10mm_Pitch0.8mm_Handsolded
- U2, U3: footprint Housings_SOIC:SOIC-8_3.9x4.9mm_Pitch1.27mm -> Project:SOIC-8_3.9x4.9mm_Pitch1.27mm_Handsolded
- moved R6 10.7 mm to (143.9, 72.6)
- moved C6 5.10 mm to (133.7, 65.2), turned to 0 degrees
- moved C4 4.32 mm to (134.0, 75.9), turned to 180 degrees
- moved C7 3.54 mm to (128.3, 70.6)
- moved R9 3.52 mm to (164.6, 53.1)
- moved J3 3.31 mm to (146.1, 53.3), turned to 270 degrees
- moved C5 2.80 mm to (139.4, 70.6)
- moved R14 2.48 mm to (163.6, 55.2)
- moved J2 2.03 mm to (138.4, 53.8)
- moved R13 1.35 mm to (163.6, 69.3)
- moved R7 1.22 mm to (163.6, 67.2)
- moved C8 1.10 mm to (163.6, 65.0)
- moved R5 1.02 mm to (130.3, 53.8)
- moved R11 1.00 mm to (162.1, 57.4)
- moved R25 0.94 mm to (174.2, 53.1)
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Connections:
- J1 pad 20: Net-(J1-Pad20) -> GND
- J2 pad 2: GND -> /TxD0
- J2 pad 3: Net-(J2-Pad3) -> GND
- J3 pad 2: Net-(J2-Pad1) -> GND
- J4 pad 3: Net-(J2-Pad3) -> Net-(J2-Pad1)
Routing:
- net +3V3: track 400.1 -> 351.5 mm, vias 10 -> 9
- net Net-(J2-Pad1): track 5.95 -> 47.1 mm
- net Net-(J2-Pad3): track 31.0 -> 0.00 mm
- net GND: track 460.8 -> 491.4 mm, vias 7 -> 11
- net Net-(J1-Pad8): track 85.4 -> 69.6 mm, vias 2 -> 4
- net /PC7: track 9.07 -> 23.9 mm
- net Net-(J1-Pad20): track 14.8 -> 0.00 mm
- net Net-(D7-Pad2): track 0.00 -> 13.2 mm, vias 0 -> 1
- net Net-(D9-Pad2): track 0.00 -> 11.9 mm, vias 0 -> 1
- net /nRE2: track 49.2 -> 38.9 mm
- net /TxD1: track 80.2 -> 73.7 mm
- net /TxD0: track 187.2 -> 181.1 mm, vias 4 -> 3
- net Net-(D8-Pad2): track 0.00 -> 4.97 mm, vias 0 -> 1
- net /PC5: track 12.5 -> 16.2 mm
- net Net-(D1-Pad2): track 6.07 -> 9.19 mm
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Other:
- outline, holes or cut-outs redrawn
- board text added: "(no RPI)"
- board text added: "+3V3"
- board text added: "3V3"
- board text added: "A"
- board text added: "B"
- board text added: "DE1"
- board text added: "DE2"
- board text added: "FTDI"
- board text added: "FTDI (J2)"
- board text added: "MISO"
- board text added: "MOSI"
- board text added: "Modbus-RTU 1"
- board text added: "Modbus-RTU 2"
- board text added: "Modbus2"
- board text added: "PA0"
- board text added: "PA1"
- board text added: "PA2"
- board text added: "PA3"
- board text added: "PA4"
- board text added: "PA5"
- board text added: "PA6"
- board text added: "PA7"
- board text added: "PB0"
- board text added: "PB1"
- board text added: "PB2"
- board text added: "PB3"
- board text added: "PC3"
- board text added: "PC4"
- board text added: "PC5"
- board text added: "PC6"
- board text added: "PC7"
- board text added: "REF"
- board text added: "RS485"
- board text added: "Raspberry"
- board text added: "Reset"
- board text added: "RxD0"
- board text added: "RxD1"
- board text added: "SCK"
- board text added: "TxD0"
- board text added: "TxD1"
- board text added: "UART0"
- board text added: "from RPI"
- board text added: "rpi-atmega324-modbus-gateway-min / V0.1 / sx"
- board text added: "~RE1~"
- board text added: "~RE2~"
- board text added: "~RST~"
- board text added: "~SS~"
- board text removed: "A B"
