File: rpi-atmega324-modbus-gateway-min/rpi-atmega324-modbus-gateway-min.sch (KiCad schematic (older format))
At the start: 26 parts, among them J1 Raspberry_Pi_2+, J16 Conn_01x11, J17 Conn_01x11, J18 Conn_01x11, J19 Conn_01x11, J2 UART-Harwin4, J3 Conn_01x02, J4 Conn_02x03_Odd_Even, J5 Atmega-ISP-6, SW1 SW_Push, U1 ATMEGA324P-20AU, Y1 12MHz

Commit message: Modbus Gateway V0.1 - Tapeout 1
Parts:
- removed J2: UART-Harwin4, Connectors_Harwin:Harwin_LTek-Male_04x2.00mm_Straight_StrainRelief, symbol UART-Harwin4
- added D7, D8, D9: LED, LEDs:LED_0805_HandSoldering, symbol LED
- added J2: UART-Harwin3, Connectors_Harwin:Harwin_LTek-Male_03x2.00mm_Straight_StrainRelief, symbol UART-Harwin3
- added R27, R28, R29: 560R, Resistors_SMD:R_1206_HandSoldering, symbol R
- added SW2: SW_SPST, Project:SW-ebay-171865305033, symbol SW_SPST
- J4: footprint Pin_Headers:Pin_Header_Straight_2x03_Pitch2.54mm -> Project:Jumper_3x_2x03_Pitch2.54mm
- U1: footprint Housings_QFP:TQFP-44_10x10mm_Pitch0.8mm -> Project:TQFP-44_10x10mm_Pitch0.8mm_Handsolded
Connections:
- wire segments 156 -> 171
- no-connect marks 31 -> 30
Other:
- note added: "Power Supply for standalone without Raspberry PI"
- moved on the sheet: J3
